Commit message: Add obstacles to 2-DOF manipulator model

File: src/pyroboplan/models/two_dof_description/two_dof.urdf (robot description, URDF)
Before this commit: robot two_dof_robot, 4 links, 3 joints
Links:
- link forearm: geometry collision box size=1.0 0.1 0.1; visual box size=1.0 0.1 0.1
- link upperarm: geometry collision box size=1.0 0.1 0.1; visual box size=1.0 0.1 0.1
