Commit message: Add whole-body differential IK example

File: src/pyroboplan/models/ur5_description/urdf/ur5_gripper.urdf (robot description, URDF)
Before this commit: robot ur5, 11 links, 10 joints
Links:
- link base_link: geometry collision mesh filename=package://ur5_description/meshes/collision/base.stl; visual mesh filename=package://ur5_description/meshes/visual/base.dae
- link forearm_link: geometry collision mesh filename=package://ur5_description/meshes/collision/forearm.stl; visual mesh filename=package://ur5_description/meshes/visual/forearm.dae
- link shoulder_link: geometry collision mesh filename=package://ur5_description/meshes/collision/shoulder.stl; visual mesh filename=package://ur5_description/meshes/visual/shoulder.dae
- link upper_arm_link: geometry collision mesh filename=package://ur5_description/meshes/collision/upperarm.stl; visual mesh filename=package://ur5_description/meshes/visual/upperarm.dae
- link wrist_1_link: geometry collision mesh filename=package://ur5_description/meshes/collision/wrist1.stl; visual mesh filename=package://ur5_description/meshes/visual/wrist1.dae
- link wrist_2_link: geometry collision mesh filename=package://ur5_description/meshes/collision/wrist2.stl; visual mesh filename=package://ur5_description/meshes/visual/wrist2.dae
- link wrist_3_link: geometry collision mesh filename=package://ur5_description/meshes/collision/wrist3.stl; visual mesh filename=package://ur5_description/meshes/visual/wrist3.dae
