Commit message: Fix models as well

File: src/pyroboplan/models/robot_12dof_description/urdf/robot_12dof.urdf (robot description, URDF)
Before this commit: robot robot_12dof, 13 links, 12 joints
Links:
- link link0: geometry collision mesh filename=package://robot_12dof_description/meshes/collision/link.dae; visual mesh filename=package://robot_12dof_description/meshes/visual/link.dae
- link link1: geometry collision mesh filename=package://robot_12dof_description/meshes/collision/link.dae; visual mesh filename=package://robot_12dof_description/meshes/visual/link.dae
- link link10: geometry collision mesh filename=package://robot_12dof_description/meshes/collision/link.dae; visual mesh filename=package://robot_12dof_description/meshes/visual/link.dae
- link link11: geometry collision mesh filename=package://robot_12dof_description/meshes/collision/link.dae; visual mesh filename=package://robot_12dof_description/meshes/visual/link.dae
- link link2: geometry collision mesh filename=package://robot_12dof_description/meshes/collision/link.dae; visual mesh filename=package://robot_12dof_description/meshes/visual/link.dae
- link link3: geometry collision mesh filename=package://robot_12dof_description/meshes/collision/link.dae; visual mesh filename=package://robot_12dof_description/meshes/visual/link.dae
- link link4: geometry collision mesh filename=package://robot_12dof_description/meshes/collision/link.dae; visual mesh filename=package://robot_12dof_description/meshes/visual/link.dae
- link link5: geometry collision mesh filename=package://robot_12dof_description/meshes/collision/link.dae; visual mesh filename=package://robot_12dof_description/meshes/visual/link.dae
- link link6: geometry collision mesh filename=package://robot_12dof_description/meshes/collision/link.dae; visual mesh filename=package://robot_12dof_description/meshes/visual/link.dae
- link link7: geometry collision mesh filename=package://robot_12dof_description/meshes/collision/link.dae; visual mesh filename=package://robot_12dof_description/meshes/visual/link.dae
- link link8: geometry collision mesh filename=package://robot_12dof_description/meshes/collision/link.dae; visual mesh filename=package://robot_12dof_description/meshes/visual/link.dae
- link link9: geometry collision mesh filename=package://robot_12dof_description/meshes/collision/link.dae; visual mesh filename=package://robot_12dof_description/meshes/visual/link.dae
