Commit message: Addresses UR5 model display issue (#79)

File: src/pyroboplan/models/ur_description/urdf/ur10_gripper.urdf (robot description, URDF)
Before this commit: robot ur5, 11 links, 10 joints
Links:
- link base: mass 0 -> 0.0
- link base_link: geometry collision mesh filename=package://ur_description/meshes/ur10/collision/base.stl; visual mesh filename=package://ur_description/meshes/ur10/visual/base.dae
- link ee_link: mass 0 -> 0.0
- link forearm_link: mass 2.275 -> 3.87; geometry collision mesh filename=package://ur_description/meshes/ur10/collision/forearm.stl; visual mesh filename=package://ur_description/meshes/ur10/visual/forearm.dae
- link shoulder_link: mass 3.7 -> 7.778; geometry collision mesh filename=package://ur_description/meshes/ur10/collision/shoulder.stl; visual mesh filename=package://ur_description/meshes/ur10/visual/shoulder.dae
- link upper_arm_link: mass 8.393 -> 12.93; geometry collision mesh filename=package://ur_description/meshes/ur10/collision/upperarm.stl; visual mesh filename=package://ur_description/meshes/ur10/visual/upperarm.dae
- link wrist_1_link: mass 1.219 -> 1.96; geometry collision mesh filename=package://ur_description/meshes/ur10/collision/wrist1.stl; visual mesh filename=package://ur_description/meshes/ur10/visual/wrist1.dae
- link wrist_2_link: mass 1.219 -> 1.96; geometry collision mesh filename=package://ur_description/meshes/ur10/collision/wrist2.stl; visual mesh filename=package://ur_description/meshes/ur10/visual/wrist2.dae
- link wrist_3_link: mass 0.1879 -> 0.202; geometry collision mesh filename=package://ur_description/meshes/ur10/collision/wrist3.stl; visual mesh filename=package://ur_description/meshes/ur10/visual/wrist3.dae
Joints:
- joint base_link-base_fixed_joint: origin xyz=0 0 0 rpy=0 0 -3.14159265 -> xyz=0 0 0 rpy=0 0 -3.14159265359
- joint ee_fixed_joint: origin xyz=0.0 0.0823 0.0 rpy=0.0 0.0 1.570796325 -> xyz=0.0 0.0922 0.0 rpy=0.0 0.0 1.57079632679
- joint elbow_joint: limit lower=-3.14159265 upper=3.14159265 effort=150.0 velocity=3.15 -> lower=-3.14159265359 upper=3.14159265359 effort=150.0 velocity=3.15; origin xyz=0.0 -0.1197 0.425 rpy=0.0 0.0 0.0 -> xyz=0.0 -0.1719 0.612 rpy=0.0 0.0 0.0
- joint shoulder_lift_joint: limit lower=-3.14159265 upper=3.14159265 effort=150.0 velocity=3.15 -> lower=-6.28318530718 upper=6.28318530718 effort=330.0 velocity=2.16; origin xyz=0.0 0.13585 0.0 rpy=0.0 1.570796325 0.0 -> xyz=0.0 0.220941 0.0 rpy=0.0 1.57079632679 0.0
- joint shoulder_pan_joint: limit lower=-3.14159265 upper=3.14159265 effort=150.0 velocity=3.15 -> lower=-6.28318530718 upper=6.28318530718 effort=330.0 velocity=2.16; origin xyz=0.0 0.0 0.089159 rpy=0.0 0.0 0.0 -> xyz=0.0 0.0 0.1273 rpy=0.0 0.0 0.0
- joint wrist_1_joint: limit lower=-3.14159265 upper=3.14159265 effort=28.0 velocity=3.2 -> lower=-6.28318530718 upper=6.28318530718 effort=54.0 velocity=3.2; origin xyz=0.0 0.0 0.39225 rpy=0.0 1.570796325 0.0 -> xyz=0.0 0.0 0.5723 rpy=0.0 1.57079632679 0.0
- joint wrist_2_joint: limit lower=-3.14159265 upper=3.14159265 effort=28.0 velocity=3.2 -> lower=-6.28318530718 upper=6.28318530718 effort=54.0 velocity=3.2; origin xyz=0.0 0.093 0.0 rpy=0.0 0.0 0.0 -> xyz=0.0 0.1149 0.0 rpy=0.0 0.0 0.0
- joint wrist_3_joint: limit lower=-3.14159265 upper=3.14159265 effort=28.0 velocity=3.2 -> lower=-6.28318530718 upper=6.28318530718 effort=54.0 velocity=3.2; origin xyz=0.0 0.0 0.09465 rpy=0.0 0.0 0.0 -> xyz=0.0 0.0 0.1157 rpy=0.0 0.0 0.0

File: src/pyroboplan/models/ur_description/urdf/ur5_on_base.urdf (robot description, URDF)
Before this commit: robot ur5_on_base, 14 links, 13 joints
Links:
- link base_link: geometry collision mesh filename=package://ur_description/meshes/ur5/collision/base.stl; visual mesh filename=package://ur_description/meshes/ur5/visual/base.dae
- link forearm_link: geometry collision mesh filename=package://ur_description/meshes/ur5/collision/forearm.stl; visual mesh filename=package://ur_description/meshes/ur5/visual/forearm.dae
- link shoulder_link: geometry collision mesh filename=package://ur_description/meshes/ur5/collision/shoulder.stl; visual mesh filename=package://ur_description/meshes/ur5/visual/shoulder.dae
- link upper_arm_link: geometry collision mesh filename=package://ur_description/meshes/ur5/collision/upperarm.stl; visual mesh filename=package://ur_description/meshes/ur5/visual/upperarm.dae
- link wrist_1_link: geometry collision mesh filename=package://ur_description/meshes/ur5/collision/wrist1.stl; visual mesh filename=package://ur_description/meshes/ur5/visual/wrist1.dae
- link wrist_2_link: geometry collision mesh filename=package://ur_description/meshes/ur5/collision/wrist2.stl; visual mesh filename=package://ur_description/meshes/ur5/visual/wrist2.dae
- link wrist_3_link: geometry collision mesh filename=package://ur_description/meshes/ur5/collision/wrist3.stl; visual mesh filename=package://ur_description/meshes/ur5/visual/wrist3.dae
