Commit message: Use Pink implementation and fill out sphere Panda model

File: src/pyroboplan/models/panda_description/urdf/panda_spheres.urdf (robot description, URDF)
Before this commit: robot panda, 12 links, 11 joints
Links:
- link panda_hand: geometry collision sphere radius=0.055; collision sphere radius=0.055
- link panda_leftfinger: geometry collision sphere radius=0.025; visual mesh filename=package://panda_description/meshes/visual/finger.dae
- link panda_link0: geometry collision sphere radius=0.1; visual mesh filename=package://panda_description/meshes/visual/link0.dae
- link panda_link1: geometry collision sphere radius=0.075; visual mesh filename=package://panda_description/meshes/visual/link1.dae
- link panda_link3: geometry collision sphere radius=0.075; collision sphere radius=0.075
- link panda_link5: geometry collision sphere radius=0.075; visual mesh filename=package://panda_description/meshes/visual/link5.dae
- link panda_rightfinger: geometry collision sphere radius=0.025; visual mesh filename=package://panda_description/meshes/visual/finger.dae

Commit message: More fixes

File: src/pyroboplan/models/panda_description/urdf/panda_spheres.urdf (robot description, URDF)
Before this commit: robot panda, 12 links, 11 joints
Links:
- link panda_link2: geometry collision sphere radius=0.075; collision sphere radius=0.075
- link panda_link3: geometry collision sphere radius=0.075; collision sphere radius=0.075
- link panda_link5: geometry collision sphere radius=0.075; collision sphere radius=0.075
- link panda_link6: geometry collision sphere radius=0.075; collision sphere radius=0.075
